File: Hardware/BAS_Hardware/BAS_Hardware.kicad_sch (KiCad schematic)
At the start: 42 parts, among them J1 Screw_Terminal_01x04, J2 Screw_Terminal_01x02, J3 Screw_Terminal_01x08, J4 Screw_Terminal_01x02, J5 Screw_Terminal_01x04, J6 Screw_Terminal_01x03, J7 Screw_Terminal_01x03, J8 Screw_Terminal_01x07, J9 Screw_Terminal_01x07, Q1 2N3904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

Commit message: add
Parts:
- removed J3: Screw_Terminal_01x08, symbol Connector:Screw_Terminal_01x08
- added C2: 330uF, EEUFS1H221LB:CAPPRD500W60D800H2000, symbol EEUFS1H221LB:EEUFS1H221LB
- added J10, J11: Screw_Terminal_01x02, TerminalBlock:TerminalBlock_bornier-2_P5.08mm, symbol Connector:Screw_Terminal_01x02
- added J12: Screw_Terminal_01x04, voltg_mini_module:Untitled, symbol Connector:Screw_Terminal_01x04
- added J2, J4: Screw_Terminal_01x04, TerminalBlock:TerminalBlock_bornier-4_P5.08mm, symbol Connector:Screw_Terminal_01x04
- added Power1: Screw_Terminal_01x02, TerminalBlock_Dinkle:TerminalBlock_Dinkle_DT-55-B01X-02_P10.00mm, symbol Connector:Screw_Terminal_01x02
- added R10, R9: 20K, Resistor_SMD:R_0805_2012Metric, symbol Device:R
- added R11: 120, Resistor_SMD:R_0805_2012Metric, symbol Device:R
- added RS485: Screw_Terminal_01x03, TerminalBlock:TerminalBlock_bornier-3_P5.08mm, symbol Connector:Screw_Terminal_01x03
- added S1: MINI-SPDT-SW, MINI-SPDT-SW:SW_MINI-SPDT-SW, symbol MINI-SPDT-SW:MINI-SPDT-SW
- added U1: MAX485E, Package_SO:SOIC-8_3.9x4.9mm_P1.27mm, symbol Interface_UART:MAX485E
- J1, J5: footprint (none) -> TerminalBlock:TerminalBlock_bornier-4_P5.08mm
- J6, J7: footprint (none) -> TerminalBlock_Dinkle:TerminalBlock_Dinkle_DT-55-B01X-03_P10.00mm
- J8, J9: footprint (none) -> TerminalBlock_Dinkle:TerminalBlock_Dinkle_DT-55-B01X-07_P10.00mm
- R1, R2, R3, R4, R5, R6, R7, R8: footprint (none) -> Resistor_SMD:R_0805_2012Metric
- supply1: renamed from J2; footprint (none) -> TerminalBlock:TerminalBlock_bornier-2_P5.08mm
- supply2: renamed from J4; footprint (none) -> TerminalBlock:TerminalBlock_bornier-2_P5.08mm
- renumbered RELAY3 to RELAY2, RELAY2 to RELAY3
Connections:
- net 5V: now also J10.1 (Pin_1), J11.1 (Pin_1), R10.2, S1.3, U1.8 (VCC)
- net COM1: no longer J7.1 (Pin_1)
- net COM2: now also J7.1 (Pin_1)
- net GND: now also C2.N, J10.2 (Pin_2), J11.2 (Pin_2), J12.3 (Pin_3), Power1.2 (Pin_2), R9.1, RS485.3 (Pin_3), U1.5 (GND)
- net I/P1: now also J2.1 (Pin_1)
- net I/P2: now also J2.2 (Pin_2)
- net I/P3: now also J2.3 (Pin_3)
- net I/P4: now also J2.4 (Pin_4)
- net I/P5: now also J4.1 (Pin_1)
- net I/P6: now also J4.2 (Pin_2)
- net I/P7: now also J4.3 (Pin_3)
- net I/P8: now also J4.4 (Pin_4)
- net RNC1: no longer J7.3 (Pin_3)
- net RNC2: now also J7.3 (Pin_3)
- net RNC3: now also J8.2 (Pin_2)
- net RNC4: now also J8.3 (Pin_3)
- net RNC5: now also J8.4 (Pin_4)
- net RNC6: now also J8.5 (Pin_5)
- net RNC7: now also J8.6 (Pin_6)
- net RNC8: now also J8.7 (Pin_7)
- net RNO1: no longer J7.2 (Pin_2)
- net RNO2: now also J7.2 (Pin_2)
- net RNO3: no longer J8.2 (Pin_2)
- net RNO4: no longer J8.3 (Pin_3)
- net RNO5: no longer J8.4 (Pin_4)
- net RNO6: no longer J8.5 (Pin_5)
- net RNO7: no longer J8.6 (Pin_6)
- net RNO8: now also J9.7 (Pin_7)
- net RX1: now also A1.16, U1.1 (RO); no longer A1.20
- net RX3: now also A1.20; no longer A1.16
- net TX1: now also A1.17, U1.4 (DI); no longer A1.21
- net TX3: now also A1.21; no longer A1.17
- net RS485: now reaches A1.5
- net RS485: now also U1.2 (~{RE}), U1.3 (DE)
- removed net RNO78: J8.7 (Pin_7), J9.7 (Pin_7)
- new net 24V: J12.2 (Pin_2), Power1.1 (Pin_1)
- new net A: R10.1, R11.1, RS485.1 (Pin_1), U1.6 (A)
- new net B: R11.2, R9.2, RS485.2 (Pin_2), U1.7 (B)
- new net Vo: C2.P, J12.4 (Pin_4), S1.2
- new net en: J12.1 (Pin_1)
Other:
- moved on the sheet: J1, J5, J6, J7, J8, J9
