File: Hardware/AVR328/AVR328.kicad_sch (KiCad schematic)
At the start: 33 parts, among them J1 EJ508A, J2 284512-8, J3 284512-8, Q2 S9013, Q3 S9013, Q4 S9013, Q5 S9013, U1 ATMEGA328P-AU, U2 L78M05CDT, Y1 Crystal

Commit message: add
Connections:
- net ADC0: now also U1.27 (PC4); no longer U1.23 (PC0)
- net ADC1: now also U1.26 (PC3); no longer U1.24 (PC1)
- net ADC3: now also U1.24 (PC1); no longer U1.26 (PC3)
- net ADC4: now also U1.23 (PC0); no longer U1.27 (PC4)
- net IN1: now also U1.15 (PB3); no longer U1.9 (PD5)
- net IN2: now also U1.14 (PB2); no longer U1.10 (PD6)
- net IN3: now also U1.13 (PB1); no longer U1.11 (PD7)
- net OUT1: now also R9.1, U1.9 (PD5); no longer R1.1, U1.12 (PB0)
- net OUT2: now also R8.1, U1.10 (PD6); no longer R7.1, U1.13 (PB1)
- net OUT3: now also R7.1, U1.11 (PD7); no longer R8.1, U1.14 (PB2)
- net OUT4: now also R1.1, U1.12 (PB0); no longer R9.1, U1.15 (PB3)
- net OUT5: no longer names the net of U1.16 (PB4)

Commit message: add
Connections:
- net GND: now also J1.1; no longer J1.2
- net at C3.1, U2.1 (IN): now also J1.2; no longer J1.1
